Commit message: Updated the qrcode code

File: toiletcleaner/urdf/toiletcleaner.urdf (robot description, URDF)
Before this commit: robot toiletcleaner, 20 links, 19 joints
Links:
- added link camera_link2, mass 1e-5; collision box size=${camera_link2} ${camera_link2} ${camera_link2}; visual box size=${camera_link2} ${camera_link2} ${camera_link2}
Joints:
- added joint camera_joint2: type fixed, parent base_link, child camera_link2, origin xyz=0.3 0 0.34 rpy=0 0 0, axis 0 1 0
